File: ol-kicad.kicad_pcb (KiCad board)
At the start: 2 copper layers, 73.5 x 52.5 mm, 29 parts, among them J2 Conn_01x02_Pin, M1 Motor_Servo, Q1 2N7000, U1 LM358, U2 NE555P

Commit message: first
Routing:
- net GND: track 280.2 -> 256.2 mm, vias 2 -> 0
- net VCC: track 211.6 -> 214.5 mm, vias 0 -> 2
